File: game_lights_out.kicad_sch (KiCad schematic)
At the start: 103 parts, among them SW1 SW_MEC_5E, SW10 SW_MEC_5E, SW11 SW_MEC_5E, SW12 SW_MEC_5E, SW13 SW_MEC_5E, SW14 SW_MEC_5E, SW15 SW_MEC_5E, SW16 SW_MEC_5E, SW17 SW_MEC_5E, SW18 SW_MEC_5E, SW19 SW_MEC_5E, SW2 SW_MEC_5E, SW20 SW_MEC_5E, SW21 SW_MEC_5E, SW22 SW_MEC_5E, SW23 SW_MEC_5E, SW24 SW_MEC_5E, SW25 SW_MEC_5E, SW26 SW_MEC_5E, SW27 SW_MEC_5E, SW28 SW_MEC_5E, SW29 SW_MEC_5E, SW3 SW_MEC_5E, SW30 SW_MEC_5E, SW31 SW_MEC_5E, SW32 SW_MEC_5E, SW33 SW_MEC_5E, SW34 SW_MEC_5E, SW35 SW_MEC_5E, SW36 SW_MEC_5E, SW37 SW_MEC_5E, SW38 SW_MEC_5E, SW39 SW_MEC_5E, SW4 SW_MEC_5E, SW40 SW_MEC_5E, SW41 SW_MEC_5E, SW42 SW_MEC_5E, SW5 SW_MEC_5E, SW6 SW_MEC_5E, SW7 SW_MEC_5E, SW8 SW_MEC_5E, SW9 SW_MEC_5E, U1 ATmega328-P, U2 ULN2803A

Commit message: WIP - major board redesign
Parts:
- SW16, SW24, SW32, SW33, SW34, SW35, SW36, SW37, SW38, SW39, SW40, SW41, SW42, SW8: footprint kicad_footprints:SW_PUSH_6mm_H5mm -> Button_Switch_THT:SW_PUSH_6mm_H5mm
Connections:
- net SR6: now also SW16.3 (K), SW16.4 (A), SW24.3 (K), SW24.4 (A), SW32.3 (K), SW32.4 (A), SW40.3 (K), SW40.4 (A), SW41.3 (K), SW41.4 (A)
Changed lines of the file:
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@@
   (junction (at 97.79 26.67) (diameter 0) (color 0 0 0 0)
   )
+  (junction (at 46.99 92.71) (diameter 0) (color 0 0 0 0)
+  )
   (junction (at 53.34 40.64) (diameter 0) (color 0 0 0 0)
   )
@@
   (junction (at 102.87 68.58) (diameter 0) (color 0 0 0 0)
   )
+  (junction (at 64.77 96.52) (diameter 0) (color 0 0 0 0)
+  )
   (junction (at 81.28 50.8) (diameter 0) (color 0 0 0 0)
   )
@@
   (junction (at 130.81 92.71) (diameter 0) (color 0 0 0 0)
   )
+  (junction (at 46.99 96.52) (diameter 0) (color 0 0 0 0)
+  )
   (junction (at 185.42 34.29) (diameter 0) (color 0 0 0 0)
   )
@@
   (junction (at 212.09 69.85) (diameter 0) (color 0 0 0 0)
   )
+  (junction (at 64.77 92.71) (diameter 0) (color 0 0 0 0)
+  )
   (junction (at 81.28 22.86) (diameter 0) (color 0 0 0 0)
   )
@@
   (junction (at 215.9 20.32) (diameter 0) (color 0 0 0 0)
   )
+  (junction (at 81.28 96.52) (diameter 0) (color 0 0 0 0)
+  )
   (junction (at 114.3 36.83) (diameter 0) (color 0 0 0 0)
   )
@@
   (junction (at 19.05 54.61) (diameter 0) (color 0 0 0 0)
   )
+  (junction (at 97.79 96.52) (diameter 0) (color 0 0 0 0)
+  )
   (junction (at 196.85 69.85) (diameter 0) (color 0 0 0 0)
   )
@@
   (junction (at 261.62 34.29) (diameter 0) (color 0 0 0 0)
   )
+  (junction (at 97.79 92.71) (diameter 0) (color 0 0 0 0)
+  )
   (junction (at 119.38 82.55) (diameter 0) (color 0 0 0 0)
   )
@@
   (junction (at 97.79 54.61) (diameter 0) (color 0 0 0 0)
   )
+  (junction (at 114.3 96.52) (diameter 0) (color 0 0 0 0)
+  )
   (junction (at 46.99 82.55) (diameter 0) (color 0 0 0 0)
   )
@@
   (junction (at 53.34 68.58) (diameter 0) (color 0 0 0 0)
   )
+  (junction (at 114.3 92.71) (diameter 0) (color 0 0 0 0)
+  )
   (junction (at 261.62 20.32) (diameter 0) (color 0 0 0 0)
   )
@@
   (junction (at 200.66 34.29) (diameter 0) (color 0 0 0 0)
   )
+  (junction (at 81.28 92.71) (diameter 0) (color 0 0 0 0)
+  )
   (junction (at 261.62 62.23) (diameter 0) (color 0 0 0 0)
   )
@@
     (stroke (width 0) (type default))
   )
+  (wire (pts (xy 46.99 92.71) (xy 46.99 96.52))
+    (stroke (width 0) (type default))
+  )
   (wire (pts (xy 177.8 137.16) (xy 177.8 132.461))
     (stroke (width 0) (type default))
@@
     (stroke (width 0) (type default))
   )
+  (wire (pts (xy 114.3 92.71) (xy 130.81 92.71))
+    (stroke (width 0) (type default))
+  )
   (wire (pts (xy 130.81 26.67) (xy 130.81 29.21))
     (stroke (width 0) (type default))
@@
     (stroke (width 0) (type default))
   )
+  (wire (pts (xy 64.77 92.71) (xy 81.28 92.71))
+    (stroke (width 0) (type default))
+  )
   (wire (pts (xy 257.81 83.82) (xy 257.81 97.155))
     (stroke (width 0) (type default))
@@
     (stroke (width 0) (type default))
   )
+  (wire (pts (xy 46.99 92.71) (xy 64.77 92.71))
+    (stroke (width 0) (type default))
+  )
   (wire (pts (xy 30.48 96.52) (xy 30.48 92.71))
     (stroke (width 0) (type default))
@@
     (stroke (width 0) (type default))
   )
+  (wire (pts (xy 81.28 92.71) (xy 97.79 92.71))
+    (stroke (width 0) (type default))
+  )
   (wire (pts (xy 130.81 54.61) (xy 130.81 57.15))
     (stroke (width 0) (type default))
@@
     (stroke (width 0) (type default))
   )
+  (wire (pts (xy 114.3 92.71) (xy 114.3 96.52))
+    (stroke (width 0) (type default))
+  )
   (wire (pts (xy 64.77 78.74) (xy 81.28 78.74))
     (stroke (width 0) (type default))
@@
     (stroke (width 0) (type default))
   )
-  (wire (pts (xy 30.48 92.71) (xy 130.81 92.71))
+  (wire (pts (xy 97.79 92.71) (xy 114.3 92.71))
+    (stroke (width 0) (type default))
+  )
+  (wire (pts (xy 30.48 92.71) (xy 46.99 92.71))
     (stroke (width 0) (type default))
   )
@@
     (stroke (width 0) (type default))
   )
+  (wire (pts (xy 97.79 92.71) (xy 97.79 96.52))
+    (stroke (width 0) (type default))
+  )
   (wire (pts (xy 227.33 41.91) (xy 231.14 41.91))
     (stroke (width 0) (type default))
@@
     (stroke (width 0) (type default))
   )
+  (wire (pts (xy 64.77 92.71) (xy 64.77 96.52))
+    (stroke (width 0) (type default))
+  )
   (wire (pts (xy 185.42 62.23) (xy 200.66 62.23))
     (stroke (width 0) (type default))
@@
     (stroke (width 0) (type default))
   )
+  (wire (pts (xy 81.28 92.71) (xy 81.28 96.52))
+    (stroke (width 0) (type default))
+  )
   (wire (pts (xy 212.09 97.155) (xy 212.09 99.695))
     (stroke (width 0) (type default))
@@
       (effects (font (size 1.27 1.27)))
     )
-    (property "Footprint" "kicad_footprints:SW_PUSH_6mm_H5mm" (at 76.2 77.47 0)
+    (property "Footprint" "Button_Switch_THT:SW_PUSH_6mm_H5mm" (at 76.2 77.47 0)
       (effects (font (size 1.27 1.27)) hide)
     )
@@
       (effects (font (size 1.27 1.27)))
     )
-    (property "Footprint" "kicad_footprints:SW_PUSH_6mm_H5mm" (at 125.73 91.44 0)
+    (property "Footprint" "Button_Switch_THT:SW_PUSH_6mm_H5mm" (at 125.73 91.44 0)
       (effects (font (size 1.27 1.27)) hide)
     )
@@
       (effects (font (size 1.27 1.27)))
     )
-    (property "Footprint" "kicad_footprints:SW_PUSH_6mm_H5mm" (at 109.22 77.47 0)
+    (property "Footprint" "Button_Switch_THT:SW_PUSH_6mm_H5mm" (at 109.22 77.47 0)
       (effects (font (size 1.27 1.27)) hide)
     )
@@
       (effects (font (size 1.27 1.27)))
     )
-    (property "Footprint" "kicad_footprints:SW_PUSH_6mm_H5mm" (at 59.69 91.44 0)
+    (property "Footprint" "Button_Switch_THT:SW_PUSH_6mm_H5mm" (at 59.69 91.44 0)
       (effects (font (size 1.27 1.27)) hide)
     )
@@
       (effects (font (size 1.27 1.27)))
     )
-    (property "Footprint" "kicad_footprints:SW_PUSH_6mm_H5mm" (at 25.4 91.44 0)
+    (property "Footprint" "Button_Switch_THT:SW_PUSH_6mm_H5mm" (at 25.4 91.44 0)
       (effects (font (size 1.27 1.27)) hide)
     )
@@
       (effects (font (size 1.27 1.27)))
     )
-    (property "Footprint" "kicad_footprints:SW_PUSH_6mm_H5mm" (at 41.91 91.44 0)
+    (property "Footprint" "Button_Switch_THT:SW_PUSH_6mm_H5mm" (at 41.91 91.44 0)
       (effects (font (size 1.27 1.27)) hide)
     )
@@
       (effects (font (size 1.27 1.27)))
     )
-    (property "Footprint" "kicad_footprints:SW_PUSH_6mm_H5mm" (at 109.22 91.44 0)
+    (property "Footprint" "Button_Switch_THT:SW_PUSH_6mm_H5mm" (at 109.22 91.44 0)
       (effects (font (size 1.27 1.27)) hide)
     )
@@
       (effects (font (size 1.27 1.27)))
     )
-    (property "Footprint" "kicad_footprints:SW_PUSH_6mm_H5mm" (at 41.91 77.47 0)
+    (property "Footprint" "Button_Switch_THT:SW_PUSH_6mm_H5mm" (at 41.91 77.47 0)
       (effects (font (size 1.27 1.27)) hide)
     )
@@
       (effects (font (size 1.27 1.27)))
     )
-    (property "Footprint" "kicad_footprints:SW_PUSH_6mm_H5mm" (at 92.71 91.44 0)
+    (property "Footprint" "Button_Switch_THT:SW_PUSH_6mm_H5mm" (at 92.71 91.44 0)
       (effects (font (size 1.27 1.27)) hide)
     )
@@
       (effects (font (size 1.27 1.27)))
     )
-    (property "Footprint" "kicad_footprints:SW_PUSH_6mm_H5mm" (at 125.73 77.47 0)
+    (property "Footprint" "Button_Switch_THT:SW_PUSH_6mm_H5mm" (at 125.73 77.47 0)
       (effects (font (size 1.27 1.27)) hide)
     )
@@
       (effects (font (size 1.27 1.27)))
     )
-    (property "Footprint" "kicad_footprints:SW_PUSH_6mm_H5mm" (at 59.69 77.47 0)
+    (property "Footprint" "Button_Switch_THT:SW_PUSH_6mm_H5mm" (at 59.69 77.47 0)
       (effects (font (size 1.27 1.27)) hide)
     )
@@
       (effects (font (size 1.27 1.27)))
     )
-    (property "Footprint" "kicad_footprints:SW_PUSH_6mm_H5mm" (at 25.4 77.47 0)
+    (property "Footprint" "Button_Switch_THT:SW_PUSH_6mm_H5mm" (at 25.4 77.47 0)
       (effects (font (size 1.27 1.27)) hide)
     )
@@
       (effects (font (size 1.27 1.27)))
     )
-    (property "Footprint" "kicad_footprints:SW_PUSH_6mm_H5mm" (at 76.2 91.44 0)
+    (property "Footprint" "Button_Switch_THT:SW_PUSH_6mm_H5mm" (at 76.2 91.44 0)
       (effects (font (size 1.27 1.27)) hide)
     )
@@
       (effects (font (size 1.27 1.27)))
     )
-    (property "Footprint" "kicad_footprints:SW_PUSH_6mm_H5mm" (at 92.71 77.47 0)
+    (property "Footprint" "Button_Switch_THT:SW_PUSH_6mm_H5mm" (at 92.71 77.47 0)
       (effects (font (size 1.27 1.27)) hide)
     )
